File: Hardware/Vorlage ATmega2560-16AU/Vorlage ATmega2560-16AU.brd (EAGLE design)
At the start: 160 x 100 mm, 151 parts, among them IC1 CD74HC14PW, IC2 ATMEGA2560640V-8AU, IC3 SS39E, IC4 SS39E, IC5 74AC138D, IC6 XC6210B332MR, Q1 16MHz, Q10 PMV27UPER, Q2 32.768kHz, Q3 PMV27UPER, Q4 PMV27UPER, Q5 PMV27UPER, Q6 PMV27UPER, Q7 PMV27UPER, Q8 PMV27UPER, Q9 PMV27UPER, U1 LM35DZ, X1 2510-, X2 +5V, X3 2514-, X4 2510-, X5 2510-

Commit message: Schema neu angeordnet
Parts:
- added C26: 100nF, rcl:C1206
- moved R14 436.3 mm to (-130.0, -280.0)
- moved R15 432.7 mm to (-120.0, -280.0)
- moved R16 429.7 mm to (-110.0, -280.0)
- moved 3.3V 428.5 mm to (-60.0, -280.0)
- moved CC1 427.7 mm to (-50.0, -280.0)
- moved CC2 427.3 mm to (-40.0, -280.0)
- moved R28 427.1 mm to (-100.0, -280.0)
- moved F1 425.1 mm to (-90.0, -280.0)
- moved U$3 422.7 mm to (-70.0, -280.0)
- moved R11 420.7 mm to (-20.0, -270.0)
- moved R17 418.9 mm to (-120.0, -270.0)
- moved C22 415.9 mm to (-30.0, -270.0)
- moved C20 412.9 mm to (-40.0, -270.0)
- moved R12 412.3 mm to (-10.0, -270.0)
- moved C19 410.4 mm to (-50.0, -270.0)
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Connections:
- net N$32 renamed PC0
- net N$35 renamed PC1
- net N$36 renamed PC2
- net N$38 renamed PC3
- net N$41 renamed PC4
- net N$42 renamed PC5
- net N$45 renamed PA0
- net N$54 renamed PH5
- net N$62 renamed PH4
- net N$71 renamed PA1
- net N$72 renamed PA2
- net N$73 renamed PH3
- net N$74 renamed PA3
- net N$76 renamed PA4
- net N$77 renamed PA5
- net N$78 renamed PA6
- net N$79 renamed PA7
- net N$80 renamed PB0
- net N$81 renamed PB1
- net N$82 renamed PB2
- net N$83 renamed PB3
- net N$84 renamed PB4
- net N$85 renamed PB5
- net N$86 renamed PB6
- net N$87 renamed PB7
- removed net N$43: IC2.59, S11.2
- removed net N$44: IC2.60, S12.2
- new net N$32: C17.1, IC2.29, Q2.1
- new net N$35: C18.1, IC2.70, Q2.2
- net GND: now also C26.2
- net PC6: now also IC2.59, S11.2; no longer C18.1, IC2.28, Q2.2
- net PC7: now also IC2.60, S12.2; no longer C17.1, IC2.29, Q2.1
- net VCC: now also C26.1

Commit message: Quarz Q2 richtig verbunden
Connections:
- net N$35: now also IC2.28; no longer IC2.70
Changed lines of the file:
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@@
 <contactref element="C18" pad="1"/>
 <contactref element="Q2" pad="2"/>
-<contactref element="IC2" pad="70"/>
-<wire x1="-22.48" y1="41.6" x2="-95.25" y2="68.58" width="0" layer="19" extent="1-1"/>
+<contactref element="IC2" pad="28"/>
+<wire x1="-35.48" y1="30.1" x2="-95.25" y2="68.58" width="0" layer="19" extent="1-1"/>
 <wire x1="-124.19" y1="142.24" x2="-95.25" y2="68.58" width="0" layer="19" extent="1-1"/>
 </signal>
