File: Hardware/Vorlage ATmega2560-16AU/Vorlage+uCBoard+Schema.sch (EAGLE design)
At the start: 160 parts, among them IC1 CD74HC14PW, IC2 ATMEGA2560640V-8AU, IC3 SS39E, IC4 SS39E, IC5 74AC138D, IC6 XC6210B332MR, Q1 16MHz, Q10 PMV27UPER, Q2 32.768kHz, Q3 PMV27UPER, Q4 PMV27UPER, Q5 PMV27UPER, Q6 PMV27UPER, Q7 PMV27UPER, Q8 PMV27UPER, Q9 PMV27UPER, U1 LM35DZ, X1 2510-, X2 +5V, X3 2514-, X4 2510-, X5 2510-

Commit message: Neue Positionsnummer und neue Stückliste
Parts:
- removed H1, H2: blau, led:LEDCHIPLED_1206
- added D20, D21: (no value), diode:DIODE-SOD123
- D1, D2: value (none) -> blau; device diode:DIODE-SOD123 -> led:LEDCHIPLED_1206
- D16: value LED -> RGB-LED
- D17: value Gruen -> +5V Power
- JTAG: value 3220-10-0100-00 -> J3
- renumbered +5V-POWER to D17, H0 to D0, H10 to D10, H11 to D11, H12 to D12, H13 to D13, H14 to D14, H15 to D15, H3 to D3, H4 to D4, H5 to D5, H6 to D6, H7 to D7, H8 to D8, H9 to D9, IC3 to U3, IC4 to U4, RGB1 to D16, U$1 to J2, U$2 to J1, U$3 to U2
Connections:
- net N$36: now also D20.C, D21.A; no longer D1.C, D2.A
- net N$38: now also D20.A; no longer D1.A
- net N$41: now also D21.C; no longer D2.C
- net N$48: now also D2.C; no longer H2.C
- net N$58: now also D1.C; no longer H1.C
- net VCC: now also D1.A, D2.A; no longer H1.A, H2.A
